File: OpenSprinkler/zones.kicad_sch (KiCad schematic)
At the start: 112 parts, among them J1 PJ-202AH, J2 Screw_Terminal_01x02, J3 Screw_Terminal_01x03, J4 Screw_Terminal_01x02, J5 Screw_Terminal_01x01, J6 Screw_Terminal_01x16, U2 SX1509, U3 LM358

Commit message: fixing connector
Parts:
- J3: footprint TerminalBlock_WAGO:TerminalBlock_WAGO_236-503_1x03_P7.50mm_45Degree -> TerminalBlock_WAGO:TerminalBlock_WAGO_236-502_1x02_P7.50mm_45Degree; symbol Connector:Screw_Terminal_01x04 -> Connector:Screw_Terminal_01x02
Connections:
- net COMMON: no longer J3.4 (Pin_4)
- net GND: no longer J3.3 (Pin_3)
Changed lines of the file:
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@@
 	(wire
 		(pts
-			(xy 185.42 80.01) (xy 185.42 87.63)
-		)
-		(stroke
-			(width 0)
-			(type default)
-		)
-	)
-	(wire
-		(pts
 			(xy 130.81 80.01) (xy 133.35 80.01)
 		)
@@
 	(wire
 		(pts
-			(xy 185.42 80.01) (xy 186.69 80.01)
-		)
-		(stroke
-			(width 0)
-			(type default)
-		)
-	)
-	(wire
-		(pts
 			(xy 163.83 125.73) (xy 163.83 128.27)
 		)
@@
 	(wire
 		(pts
-			(xy 184.15 82.55) (xy 186.69 82.55)
-		)
-		(stroke
-			(width 0)
-			(type default)
-		)
-	)
-	(wire
-		(pts
 			(xy 151.13 72.39) (xy 151.13 82.55)
 		)
@@
 		)
 	)
-	(global_label "COMMON"
-		(shape input)
-		(at 184.15 82.55 180)
-		(fields_autoplaced yes)
-		(effects
-			(font
-				(size 1.27 1.27)
-			)
-			(justify right)
-		)
-		(property "Intersheetrefs" "${INTERSHEET_REFS}"
-			(at 173.0799 82.55 0)
-			(effects
-				(font
-					(size 1.27 1.27)
-				)
-				(justify right)
-				(hide yes)
-			)
-		)
-	)
 	(global_label "Zone 7"
 		(shape output)
@@
 	)
 	(symbol
-		(lib_id "power:GND")
-		(at 185.42 87.63 0)
-		(unit 1)
-		(exclude_from_sim no)
-		(in_bom yes)
-		(on_board yes)
-		(dnp no)
-		(fields_autoplaced yes)
-		(property "Reference" "#PWR031"
-			(at 185.42 93.98 0)
-			(effects
-				(font
-					(size 1.27 1.27)
-				)
-				(hide yes)
-			)
-		)
-		(property "Value" "GND"
-			(at 185.42 92.71 0)
-			(effects
-				(font
-					(size 1.27 1.27)
-				)
-			)
-		)
-		(property "Footprint" ""
-			(at 185.42 87.63 0)
-			(effects
-				(font
-					(size 1.27 1.27)
-				)
-				(hide yes)
-			)
-		)
-		(property "Datasheet" ""
-			(at 185.42 87.63 0)
-			(effects
-				(font
-					(size 1.27 1.27)
-				)
-				(hide yes)
-			)
-		)
-		(property "Description" "Power symbol creates a global label with name \"GND\" , ground"
-			(at 185.42 87.63 0)
-			(effects
-				(font
-					(size 1.27 1.27)
-				)
-				(hide yes)
-			)
-		)
-		(pin "1"
-		)
-		(instances
-			(project "OpenSprinkler"
-				(path "/1e7a19e7-c172-48cb-8290-979862293d8a/c3033e14-a954-4331-8f1d-87f6033f6a65"
-					(reference "#PWR031")
-					(unit 1)
-				)
-			)
-		)
-	)
-	(symbol
 		(lib_name "TVSSMB_1")
 		(lib_id "o-eagle-import:TVSSMB")
@@
 	)
 	(symbol
-		(lib_id "Connector:Screw_Terminal_01x04")
-		(at 191.77 77.47 0)
+		(lib_id "Connector:Screw_Terminal_01x02")
+		(at 191.77 74.93 0)
 		(unit 1)
 		(exclude_from_sim no)
@@
 		(dnp no)
 		(property "Reference" "J3"
-			(at 194.31 78.105 0)
+			(at 194.31 75.565 0)
 			(effects
 				(font
@@
 		)
 		(property "Value" "Screw_Terminal_01x03"
-			(at 194.31 80.645 0)
+			(at 194.31 78.105 0)
 			(effects
 				(font
@@
 			)
 		)
-		(property "Footprint" "TerminalBlock_WAGO:TerminalBlock_WAGO_236-503_1x03_P7.50mm_45Degree"
-			(at 191.77 77.47 0)
+		(property "Footprint" "TerminalBlock_WAGO:TerminalBlock_WAGO_236-502_1x02_P7.50mm_45Degree"
+			(at 191.77 74.93 0)
 			(effects
 				(font
@@
 		)
 		(property "Datasheet" "~"
-			(at 191.77 77.47 0)
+			(at 191.77 74.93 0)
 			(effects
 				(font
@@
 			)
 		)
-		(property "Description" "Generic screw terminal, single row, 01x04, script generated (kicad-library-utils/schlib/autogen/connector/)"
-			(at 191.77 77.47 0)
+		(property "Description" "Generic screw terminal, single row, 01x02, script generated (kicad-library-utils/schlib/autogen/connector/)"
+			(at 191.77 74.93 0)
 			(effects
 				(font
@@
 		(pin "2"
 		)
-		(pin "3"
-		)
-		(pin "4"
-		)
 		(instances
