File: OpenSprinkler/OpenSprinkler.kicad_pcb (KiCad board)
At the start: 2 copper layers, 207.3 x 67.7 mm, 215 parts, among them J1 PJ-202AH, J2 Screw_Terminal_01x02, J3 Screw_Terminal_01x03, J4 Screw_Terminal_01x02, J5 Screw_Terminal_01x01, J6 Screw_Terminal_01x16, Q1 MBT2222ADW1T1, U1 AP63203WU, U2 SX1509, U3 LM358, U4 M24C02-FMN, U5 ESP32-WROOM-32, U6 PCF8563TS, U7 IS31FL3236A-TQ, U8 IS31FL3236A-TQ, Y1 32.768kHz

Commit message: fixing connector
Parts:
- J3: footprint TerminalBlock_WAGO:TerminalBlock_WAGO_236-503_1x03_P7.50mm_45Degree -> TerminalBlock_WAGO:TerminalBlock_WAGO_236-502_1x02_P7.50mm_45Degree
- U2: footprint SparkFun-DigitalIC:QFN-28 -> SX1509BIULTRT:QFN40P400X400X60-29N

Commit message: Updating pcb
Routing:
- net LED9: track 50.5 -> 58.0 mm
- net LED15_1: track 32.9 -> 39.5 mm
- net LED12: track 47.9 -> 53.4 mm
- net LED21_1: track 28.3 -> 32.6 mm
- net LED19_1: track 31.9 -> 28.0 mm
- net LED33: track 63.5 -> 66.9 mm
- net LED33_1: track 52.2 -> 55.4 mm
- net LED34: track 68.5 -> 71.8 mm
- net LED20_1: track 32.1 -> 28.9 mm
- net LED4: track 57.3 -> 59.6 mm
- net LED3: track 65.3 -> 67.6 mm
- net LED5: track 61.4 -> 59.4 mm
- net LED6: track 61.2 -> 59.4 mm
- net LED12_1: track 53.5 -> 55.2 mm
- net LED29_1: track 42.8 -> 41.1 mm
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
Commit message: Updating pcb
Routing:
- net LED9_1: track 56.3 -> 59.3 mm
- net LED6_1: track 66.1 -> 68.0 mm
- net LED12_1: track 55.2 -> 56.5 mm
- net LED11_1: track 53.6 -> 52.4 mm
- net LED30: track 52.2 -> 51.1 mm
- net LED29: track 48.7 -> 47.7 mm
- net LED28: track 47.1 -> 46.1 mm
- net LED10_1: track 50.6 -> 51.5 mm
